File: schematicMain.brd (EAGLE design)
At the start: 100.3 x 100 mm, 60 parts, among them K1 G5L, K2 G5L, K3 G5L, K4 G5L, K5 G5L, Q1 MMBTA56-SOT23, Q2 MMBTA56-SOT23, Q3 MMBTA56-SOT23, Q4 MMBTA56-SOT23, Q5 MMBTA56-SOT23

Commit message: Updated Relay modules
Parts:
- removed Q1, Q2, Q3, Q4, Q5: MMBTA56-SOT23, transistor-pnp:SOT23
- removed R8: 1k, resistor:M1206
- removed X6, X7, X8: (no value), con-wago-500:W237-102
- added OK1, OK2, OK3, OK4, OK5: 4N35, optocoupler:DIL06
- added R15: 1k, resistor:M1206
- added VT1, VT2, VT3, VT4, VT5: MMBT3904LT1, transistor-npn:SOT23-BEC
- added X2, X3, X4: (no value), con-wago-500:W237-102
- moved R4 273.8 mm to (-74.9, -193.0)
- moved X1 272.7 mm to (-62.2, -174.0), turned to 0 degrees
- moved D10 261.6 mm to (-69.8, -193.0), turned to 0 degrees
- moved D11 259.1 mm to (-71.1, -186.7), turned to 0 degrees
- moved K5 248.5 mm to (-66.0, -161.3), turned to 0 degrees
- moved PWR-5 244.5 mm to (-55.9, -186.7), turned to 0 degrees
- moved R3 212.5 mm to (-53.3, -144.8)
- moved D7 211.1 mm to (-48.3, -144.8), turned to 0 degrees
- moved D8 205.7 mm to (-49.5, -138.4)
- moved PWR-4 201.8 mm to (-34.3, -138.4)
- moved K4 171.6 mm to (-44.5, -113.0), turned to 0 degrees
- moved R2 152.4 mm to (-31.8, -96.5)
- moved D5 149.9 mm to (-26.7, -96.5), turned to 0 degrees
- moved D6 144.0 mm to (-27.9, -90.2)
- moved PWR-3 140.9 mm to (-12.7, -90.2)
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Connections:
- removed net N$20 (its old number): Q3.1, R3.1
- new net N$12: D4.A, K2.2, VT2.C
- new net N$19: D5.A, OK3.4, VT3.B
- new net N$21: D11.A, K5.2, VT5.C
- new net N$26: D8.A, K4.2, VT4.C
- new net N$28: D3.A, OK2.4, VT2.B
- new net N$5: D2.A, K1.2, VT1.C
- net 5V0: now also D11.C, D2.C, D4.C, D6.C, D8.C, K1.1, K2.1, K3.1, K4.1, K5.1, OK1.5, OK2.5, OK3.5, OK4.5, OK5.5; no longer Q1.2, Q2.2, Q3.2, Q4.2, Q5.2
- net GND: now also OK1.2, OK2.2, OK3.2, OK4.2, OK5.2, VT1.E, VT2.E, VT3.E, VT4.E, VT5.E; no longer D11.A, D2.A, D4.A, D6.A, D8.A, K1.2, K2.2, K3.2, K4.2, K5.2
- net N$11: now also OK2.1, R15.1; no longer D3.A, D4.C, K2.1, Q2.3
- net N$13: now also K3.P, X3.2; no longer Q2.1, R2.1
- net N$15: now also K3.S, X3.1; no longer K3.P, X7.2
- net N$16: now also OK3.1, R2.1; no longer K3.S, X7.1
- net N$17: now also OK5.1, R4.1; no longer D10.A, D11.C, K5.1, Q5.3
- net N$18: now also D6.A, K3.2, VT3.C; no longer D5.A, D6.C, K3.1, Q3.3
- net N$22: now also X4.2; no longer X8.2
- net N$23: now also X4.1; no longer X8.1
- net N$24: now also D10.A, OK5.4, VT5.B; no longer Q5.1, R8.1
- net N$25: now also OK4.1, R3.1; no longer D7.A, D8.C, K4.1, Q4.3
- net N$27: now also D7.A, OK4.4, VT4.B; no longer Q4.1, R4.1
- net N$3: now also X2.2; no longer X6.2
- net N$4: now also OK1.4, VT1.B; no longer D2.C, K1.1, Q1.3
- net N$7: now also OK1.1; no longer Q1.1
- net N$9: now also X2.1; no longer X6.1
- net SIGNAL-RELAY-2: now also R15.2; no longer R2.2
- net SIGNAL-RELAY-3: now also R2.2; no longer R3.2
- net SIGNAL-RELAY-4: now also R3.2; no longer R4.2
- net WELCOME-SIGNAL: now also R4.2; no longer R8.2
Routing:
- net 5V0: track 566.9 -> 0.00 mm, vias 3 -> 0
- net GND: track 415.4 -> 0.00 mm, vias 1 -> 0
- net SIGNAL-RELAY-4: track 93.4 -> 0.00 mm, vias 2 -> 0
- net SIGNAL-RELAY-3: track 86.5 -> 0.00 mm
- net WELCOME-SIGNAL: track 83.7 -> 0.00 mm, vias 1 -> 0
- net SIGNAL-RELAY-2: track 74.4 -> 0.00 mm
- net GND@1: track 71.2 -> 0.00 mm
- net SIGNAL-RELAY-1: track 65.3 -> 0.00 mm
- net GND@4: track 63.7 -> 0.00 mm
- net DOOR: track 59.0 -> 0.00 mm
- net 3V3@2: track 54.0 -> 0.00 mm, vias 2 -> 0
- net PIR: track 51.6 -> 0.00 mm, vias 1 -> 0
- net S-GREEN: track 41.8 -> 0.00 mm
- net GND@2: track 40.5 -> 0.00 mm
- net S-BLUE: track 40.0 -> 0.00 mm
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
Commit message: update 23-11-2018
Parts:
- D9: device SparkFun-LED:PLCC-6-LED -> SparkFun-LED:LED-TRICOLOR-5050
- moved H2 78.3 mm to (92.7, 27.9)
- moved H3 28.4 mm to (88.9, 82.5)
- moved D2 26.7 mm to (36.8, 35.6)
- moved D1 21.7 mm to (25.4, 45.7)
- moved R1 21.6 mm to (34.3, 44.5)
- moved PWR-2 19.1 mm to (31.8, 39.4)
- moved H4 11.4 mm to (11.4, 76.2)
- moved X5 2.84 mm to (5.08, 5.08)
- moved D9 2.84 mm to (95.2, 77.5), turned to 0 degrees
- moved R10 1.27 mm to (49.5, 54.6)
- moved R11 1.27 mm to (43.2, 54.6)
- moved R12 1.27 mm to (36.8, 54.6)
- moved R13 1.27 mm to (30.5, 54.6)
- moved R14 1.27 mm to (24.1, 54.6)
- moved R9 1.27 mm to (55.9, 54.6)
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Connections:
- net GND@1: now also D9.4, D9.5, D9.6; no longer D9.CB, D9.CG, D9.CR
- net S-BLUE: now also D9.3; no longer D9.AB
- net S-GREEN: now also D9.1; no longer D9.AG
- net S-RED: now also D9.2; no longer D9.AR
Routing:
- net GND: track 0.00 -> 125.0 mm
- net 5V0: track 0.00 -> 110.3 mm

Commit message: Pcb design finished
Parts:
- removed D11, D4, D6, D8: 1N4148DO35-10, diode:DO35-10
- removed X1: (no value), con-wago-500:W237-102
- added D12, D13, D14, D15: (no value), diode:SOD80C
- added WELCOME: (no value), con-wago-500:W237-102
- D2: value 1N4148DO35-10 -> (none); device diode:DO35-10 -> diode:SOD80C
- moved R4 287.8 mm to (83.8, 47.0), turned to 90 degrees
- moved D10 279.7 mm to (83.8, 40.6), turned to 90 degrees
- moved PWR-5 268.8 mm to (87.6, 40.6), turned to 270 degrees
- moved OK5 266.0 mm to (77.5, 43.2), turned to 180 degrees
- moved VT5 250.4 mm to (82.5, 35.6), turned to 270 degrees
- moved K5 233.8 mm to (81.3, 20.3), turned to 270 degrees
- moved R3 225.9 mm to (66.0, 47.0), turned to 90 degrees
- moved D7 217.8 mm to (66.0, 40.6), turned to 90 degrees
- moved PWR-4 207.2 mm to (69.8, 40.6), turned to 270 degrees
- moved OK4 204.0 mm to (59.7, 43.2), turned to 180 degrees
- moved VT4 188.6 mm to (64.8, 35.6), turned to 270 degrees
- moved K4 171.6 mm to (63.5, 20.3), turned to 270 degrees
- moved R2 164.3 mm to (48.3, 47.0), turned to 90 degrees
- moved X4 158.2 mm to (48.3, 5.08)
- moved D5 156.3 mm to (48.3, 40.6), turned to 90 degrees
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- renumbered DOOR to -DOOR+, PIR to GND-PIR-5V, U$2 to DHT11
Connections:
- net 5V0: now also D12.C, D13.C, D14.C, D15.C; no longer D11.C, D4.C, D6.C, D8.C
- net N$10: now also WELCOME.1; no longer X1.1
- net N$12: now also D2.A; no longer D4.A
- net N$18: now also D13.A; no longer D6.A
- net N$21: now also D15.A; no longer D11.A
- net N$26: now also D14.A; no longer D8.A
- net N$5: now also D12.A; no longer D2.A
- net N$6: now also WELCOME.2; no longer X1.2
Routing:
- net 5V0: track 110.3 -> 558.1 mm, vias 0 -> 2
- net GND: track 125.0 -> 353.3 mm, vias 0 -> 10
- net SIGNAL-RELAY-4: track 0.00 -> 88.1 mm
- net SIGNAL-RELAY-3: track 0.00 -> 78.2 mm
- net GND@1: track 0.00 -> 69.5 mm
- net SIGNAL-RELAY-2: track 0.00 -> 68.2 mm
- net PIR: track 0.00 -> 61.7 mm, vias 0 -> 4
- net SIGNAL-RELAY-1: track 0.00 -> 58.2 mm
- net DOOR: track 0.00 -> 57.6 mm
- net GND@4: track 0.00 -> 55.5 mm, vias 0 -> 1
- net 3V3@2: track 0.00 -> 51.2 mm
- net S-GREEN: track 0.00 -> 41.2 mm
- net N$6: track 0.00 -> 40.1 mm
- net S-BLUE: track 0.00 -> 38.9 mm
- net GND@2: track 0.00 -> 38.5 mm
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