File: schematicMain.sch (EAGLE design)
At the start: 60 parts, among them K1 G5L, K2 G5L, K3 G5L, K4 G5L, K5 G5L, Q1 MMBTA56-SOT23, Q2 MMBTA56-SOT23, Q3 MMBTA56-SOT23, Q4 MMBTA56-SOT23, Q5 MMBTA56-SOT23

Commit message: Updated Relay modules
Parts:
- removed Q1, Q2, Q3, Q4, Q5: MMBTA56-SOT23, transistor-pnp:MMBTA56-SOT23
- removed R8: 1k, resistor:R-US_M1206
- removed X6, X7, X8: (no value), con-wago-500:W237-102
- added OK1, OK2, OK3, OK4, OK5: 4N35, optocoupler:4N35
- added R15: 1k, resistor:R-US_M1206
- added VT1, VT2, VT3, VT4, VT5: MMBT3904LT1, transistor-npn:MMBT3904LT1
- added X2, X3, X4: (no value), con-wago-500:W237-102
Connections:
- removed net N$20 (its old number): Q3.B, R3.1
- new net N$12: D4.A, K21.2, VT2.C
- new net N$19: D5.A, OK3.EMI, VT3.B
- new net N$21: D11.A, K51.2, VT5.C
- new net N$26: D8.A, K41.2, VT4.C
- new net N$28: D3.A, OK2.EMI, VT2.B
- new net N$5: D2.A, K11.2, VT1.C
- net 5V0: now also D11.C, D2.C, D4.C, D6.C, D8.C, K11.1, K21.1, K31.1, K41.1, K51.1, OK1.COL, OK2.COL, OK3.COL, OK4.COL, OK5.COL; no longer Q1.E, Q2.E, Q3.E, Q4.E, Q5.E
- net GND: now also OK1.C, OK2.C, OK3.C, OK4.C, OK5.C, VT1.E, VT2.E, VT3.E, VT4.E, VT5.E; no longer D11.A, D2.A, D4.A, D6.A, D8.A, K11.2, K21.2, K31.2, K41.2, K51.2
- net N$11: now also OK2.A, R15.1; no longer D3.A, D4.C, K21.1, Q2.C
- net N$13: now also K32.P, X3-2.KL; no longer Q2.B, R2.1
- net N$15: now also K32.S, X3-1.KL; no longer K32.P, X7-2.KL
- net N$16: now also OK3.A, R2.1; no longer K32.S, X7-1.KL
- net N$17: now also OK5.A, R4.1; no longer D10.A, D11.C, K51.1, Q5.C
- net N$18: now also D6.A, K31.2, VT3.C; no longer D5.A, D6.C, K31.1, Q3.C
- net N$22: now also X4-2.KL; no longer X8-2.KL
- net N$23: now also X4-1.KL; no longer X8-1.KL
- net N$24: now also D10.A, OK5.EMI, VT5.B; no longer Q5.B, R8.1
- net N$25: now also OK4.A, R3.1; no longer D7.A, D8.C, K41.1, Q4.C
- net N$27: now also D7.A, OK4.EMI, VT4.B; no longer Q4.B, R4.1
- net N$3: now also X2-2.KL; no longer X6-2.KL
- net N$4: now also OK1.EMI, VT1.B; no longer D2.C, K11.1, Q1.C
- net N$7: now also OK1.A; no longer Q1.B
- net N$9: now also X2-1.KL; no longer X6-1.KL
- net SIGNAL-RELAY-2: now also R15.2; no longer R2.2
- net SIGNAL-RELAY-3: now also R2.2; no longer R3.2
- net SIGNAL-RELAY-4: now also R3.2; no longer R4.2
- net WELCOME-SIGNAL: now also R4.2; no longer R8.2
Other:
- moved on the sheet: D1, D10, D11, D2, D3, D4, D5, D6, D7, D8, K1, K2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

Commit message: update 23-11-2018
Parts:
- D9: device SparkFun-LED:LED-RGBPLCC-6 -> SparkFun-LED:LED-RGBNO_IC
Changed lines of the file:
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@@
 <part name="U$1" library="RPI-Zero" deviceset="RPI-ZERO" device=""/>
 <part name="U$2" library="diy-modules" deviceset="TEMP-HUM-SENSOR-DHT11" device=""/>
-<part name="D9" library="SparkFun-LED" library_urn="urn:adsk.eagle:library:529" deviceset="LED-RGB" device="PLCC-6" package3d_urn="urn:adsk.eagle:package:39373/1" value="RGB"/>
+<part name="D9" library="SparkFun-LED" library_urn="urn:adsk.eagle:library:529" deviceset="LED-RGB" device="NO_IC" package3d_urn="urn:adsk.eagle:package:39374/1" value="RGB"/>
 <part name="PIR" library="con-wago-500" library_urn="urn:adsk.eagle:library:195" deviceset="W237-103" device="" package3d_urn="urn:adsk.eagle:package:10691/1"/>
 <part name="DOOR" library="con-wago-500" library_urn="urn:adsk.eagle:library:195" deviceset="W237-102" device="" package3d_urn="urn:adsk.eagle:package:10688/1"/>
@@
 <instance part="D9" gate="G$1" x="22.86" y="104.14" smashed="yes" rot="R90">
 <attribute name="NAME" x="17.145" y="104.14" size="1.778" layer="95" font="vector" rot="R90" align="bottom-center"/>
-<attribute name="VALUE" x="28.575" y="104.14" size="1.778" layer="95" font="vector" rot="R90" align="top-center"/>
 </instance>
 <instance part="PIR" gate="-1" x="55.88" y="137.16" smashed="yes" rot="R270">

Commit message: Pcb design finished
Parts:
- removed D11, D4, D6, D8: 1N4148DO35-10, diode:1N4148DO35-10
- added D12, D13, D14, D15: (no value), diode:DIODE-SOD80C
- D2: value 1N4148DO35-10 -> (none); device diode:1N4148DO35-10 -> diode:DIODE-SOD80C
- renumbered DOOR to -DOOR+, PIR to GND-PIR-5V, U$2 to DHT11, X1 to WELCOME
Connections:
- net 5V0: now also D12.C, D13.C, D14.C, D15.C; no longer D11.C, D4.C, D6.C, D8.C
- net N$12: now also D2.A; no longer D4.A
- net N$18: now also D13.A; no longer D6.A
- net N$21: now also D15.A; no longer D11.A
- net N$26: now also D14.A; no longer D8.A
- net N$5: now also D12.A; no longer D2.A
Other:
- moved on the sheet: D2
